File: schematics/kicad/rev1.2/midi-viscount-rte0616.kicad_pcb (KiCad board)
At the start: 2 copper layers, 95 x 50.8 mm, 21 parts, among them J1 Conn_02x07_Odd_Even, J10 Conn_01x01_Pin, J11 Conn_01x01_Pin, J12 Conn_01x01_Pin, J13 Conn_01x01_Pin, J2 Conn_01x01_Pin, J3 Conn_01x01_Pin, J4 Conn_01x01_Pin, J5 Conn_01x01_Pin, J6 Conn_01x01_Pin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

Commit message: Update docs
Update docs
Parts:
- removed the REF** at (47.6, 81.6)
- removed the REF** at (47.6, 39.0)
- removed the REF** at (134.4, 81.6)
- removed the REF** at (134.4, 39.0)
- added REF**: MountingHole_3.2mm_M3_ISO7380, MountingHole:MountingHole_3.2mm_M3_ISO7380, F.Cu at (47.6, 39.0)
- added REF**: MountingHole_3.2mm_M3_ISO7380, MountingHole:MountingHole_3.2mm_M3_ISO7380, F.Cu at (134.4, 39.0)
- added REF**: MountingHole_3.2mm_M3_ISO7380, MountingHole:MountingHole_3.2mm_M3_ISO7380, F.Cu at (134.4, 81.6)
- added REF**: MountingHole_3.2mm_M3_ISO7380, MountingHole:MountingHole_3.2mm_M3_ISO7380, F.Cu at (47.6, 81.6)
